Commit message: Update elbow joint limit in human model (different from 0)

File: urdf/human_model.urdf (robot description, URDF)
Before this commit: robot hooman, 45 links, 44 joints
Joints:
- joint left_elbow_flexion: limit lower=0.0 upper=2.47836753783 effort=75.0 velocity=1.0 -> lower=-0.087 upper=2.47836753783 effort=75.0 velocity=1.0
- joint right_elbow_flexion: limit lower=0.0 upper=2.47836753783 effort=75.0 velocity=1.0 -> lower=-0.087 upper=2.47836753783 effort=75.0 velocity=1.0

File: urdf/human_model_fixed_base.urdf (robot description, URDF)
Before this commit: robot hooman, 46 links, 45 joints
Joints:
- joint left_elbow_flexion: limit lower=0.0 upper=2.47836753783 effort=75.0 velocity=1.0 -> lower=-0.087 upper=2.47836753783 effort=75.0 velocity=1.0
- joint right_elbow_flexion: limit lower=0.0 upper=2.47836753783 effort=75.0 velocity=1.0 -> lower=-0.087 upper=2.47836753783 effort=75.0 velocity=1.0

File: xacro/dhm43_ISB.xacro (robot description, xacro)
@@ -675,5 +675,5 @@
 		<axis xyz="0 0 1"/>
 		<origin xyz="0 ${-shoulder_elbow} 0"/>
-		<limit effort="${75*forceCapacity}" lower="${-0*PI/180}" upper="${142*PI/180}" velocity="${maxVelJoint}"/>
+		<limit effort="${75*forceCapacity}" lower="${-5*PI/180}" upper="${142*PI/180}" velocity="${maxVelJoint}"/>
 		<dynamics damping="${jointDamping}" friction="${jointFriction}"/>
 	</joint>
@@ -748,5 +748,5 @@
 		<axis xyz="0 0 1"/>
 		<origin xyz="0 ${-shoulder_elbow} 0"/>
-		<limit effort="${75*forceCapacity}" lower="${-0*PI/180}" upper="${142*PI/180}" velocity="${maxVelJoint}"/>
+		<limit effort="${75*forceCapacity}" lower="${-5*PI/180}" upper="${142*PI/180}" velocity="${maxVelJoint}"/>
 		<dynamics damping="${jointDamping}" friction="${jointFriction}"/>
 	</joint>

File: xacro/human_model.xacro (robot description, xacro)
@@ -675,5 +675,5 @@
 		<axis xyz="0 0 1"/>
 		<origin xyz="0 ${-shoulder_elbow} 0"/>
-		<limit effort="${75*forceCapacity}" lower="${-0*PI/180}" upper="${142*PI/180}" velocity="${maxVelJoint}"/>
+		<limit effort="${75*forceCapacity}" lower="${-5*PI/180}" upper="${142*PI/180}" velocity="${maxVelJoint}"/>
 		<dynamics damping="${jointDamping}" friction="${jointFriction}"/>
 	</joint>
@@ -748,5 +748,5 @@
 		<axis xyz="0 0 1"/>
 		<origin xyz="0 ${-shoulder_elbow} 0"/>
-		<limit effort="${75*forceCapacity}" lower="${-0*PI/180}" upper="${142*PI/180}" velocity="${maxVelJoint}"/>
+		<limit effort="${75*forceCapacity}" lower="${-5*PI/180}" upper="${142*PI/180}" velocity="${maxVelJoint}"/>
 		<dynamics damping="${jointDamping}" friction="${jointFriction}"/>
 	</joint>

Commit message: Update human model with higher inertia for "virtual" bodies. Test joint order

File: urdf/human_model.urdf (robot description, URDF)
Before this commit: robot hooman, 45 links, 44 joints
Links:
- link body_C1: mass 0.001 -> 0.1
- link body_C7_1: mass 0.001 -> 0.1
- link body_C7_2: mass 0.001 -> 0.1
- link body_CSJ_left_clavicular: mass 0.001 -> 0.1
- link body_CSJ_right_clavicular: mass 0.001 -> 0.1
- link body_L5_1: mass 0.001 -> 0.1
- link body_L5_2: mass 0.001 -> 0.1
- link body_T12_1: mass 0.001 -> 0.1
- link body_T12_2: mass 0.001 -> 0.1
- link body_left_ankle: mass 0.001 -> 0.1
- link body_left_elbow: mass 0.001 -> 0.1
- link body_left_hip_1: mass 0.001 -> 0.1
- link body_left_hip_2: mass 0.001 -> 0.1
- link body_left_knee: mass 0.001 -> 0.1
- link body_left_shoulder_1: mass 0.001 -> 0.1
- link body_left_shoulder_2: mass 0.001 -> 0.1
- link body_left_wrist: mass 0.001 -> 0.1
- link body_right_ankle: mass 0.001 -> 0.1
- link body_right_elbow: mass 0.001 -> 0.1
- link body_right_hip_1: mass 0.001 -> 0.1
- link body_right_hip_2: mass 0.001 -> 0.1
- link body_right_knee: mass 0.001 -> 0.1
- link body_right_shoulder_1: mass 0.001 -> 0.1
- link body_right_shoulder_2: mass 0.001 -> 0.1
- link body_right_wrist: mass 0.001 -> 0.1
- link head: mass 4.34506412008 -> 4.18602407037
- link left_arm: mass 1.74495037103 -> 1.68108088923
- link left_clavicular: mass 0.518326492016 -> 0.499354465648
- link left_foot: mass 0.910491316081 -> 0.877165091159
- link left_forearm: mass 1.06160792958 -> 1.02275046437
- link left_hand: mass 0.41408646156 -> 0.398929877075
- link left_shank: mass 2.80920246717 -> 2.70637873715
- link left_thigh: mass 9.16927117713 -> 8.83365326597
- link lumbar_spine: mass 10.4080382663 -> 10.0270784284
- link neck: mass 0.482784902231 -> 0.465113785597
- link pelvis: mass 7.15341845835 -> 6.89158572223
- link right_arm: mass 1.74495037103 -> 1.68108088923
- link right_clavicular: mass 0.518326492016 -> 0.499354465648
- link right_foot: mass 0.910491316081 -> 0.877165091159
- link right_forearm: mass 1.06160792958 -> 1.02275046437
- link right_hand: mass 0.41408646156 -> 0.398929877075
- link right_shank: mass 2.80920246717 -> 2.70637873715
- link right_thigh: mass 9.16927117713 -> 8.83365326597
- link root: mass 0.001 -> 0.1
- link thoracic_spine: mass 9.32987685629 -> 8.98838038167
Joints:
- joint left_elbow_flexion: limit lower=-0.087 upper=2.47836753783 effort=75.0 velocity=1.0 -> lower=-0.0872664625997 upper=2.47836753783 effort=75.0 velocity=1.0
- joint right_elbow_flexion: limit lower=-0.087 upper=2.47836753783 effort=75.0 velocity=1.0 -> lower=-0.0872664625997 upper=2.47836753783 effort=75.0 velocity=1.0

File: urdf/human_model_fixed_base.urdf (robot description, URDF)
Before this commit: robot hooman, 46 links, 45 joints
Links:
- link body_C1: mass 0.001 -> 0.1
- link body_C7_1: mass 0.001 -> 0.1
- link body_C7_2: mass 0.001 -> 0.1
- link body_CSJ_left_clavicular: mass 0.001 -> 0.1
- link body_CSJ_right_clavicular: mass 0.001 -> 0.1
- link body_L5_1: mass 0.001 -> 0.1
- link body_L5_2: mass 0.001 -> 0.1
- link body_T12_1: mass 0.001 -> 0.1
- link body_T12_2: mass 0.001 -> 0.1
- link body_left_ankle: mass 0.001 -> 0.1
- link body_left_elbow: mass 0.001 -> 0.1
- link body_left_hip_1: mass 0.001 -> 0.1
- link body_left_hip_2: mass 0.001 -> 0.1
- link body_left_knee: mass 0.001 -> 0.1
- link body_left_shoulder_1: mass 0.001 -> 0.1
- link body_left_shoulder_2: mass 0.001 -> 0.1
- link body_left_wrist: mass 0.001 -> 0.1
- link body_right_ankle: mass 0.001 -> 0.1
- link body_right_elbow: mass 0.001 -> 0.1
- link body_right_hip_1: mass 0.001 -> 0.1
- link body_right_hip_2: mass 0.001 -> 0.1
- link body_right_knee: mass 0.001 -> 0.1
- link body_right_shoulder_1: mass 0.001 -> 0.1
- link body_right_shoulder_2: mass 0.001 -> 0.1
- link body_right_wrist: mass 0.001 -> 0.1
- link head: mass 4.34506412008 -> 4.18602407037
- link left_arm: mass 1.74495037103 -> 1.68108088923
- link left_clavicular: mass 0.518326492016 -> 0.499354465648
- link left_foot: mass 0.910491316081 -> 0.877165091159
- link left_forearm: mass 1.06160792958 -> 1.02275046437
- link left_hand: mass 0.41408646156 -> 0.398929877075
- link left_shank: mass 2.80920246717 -> 2.70637873715
- link left_thigh: mass 9.16927117713 -> 8.83365326597
- link lumbar_spine: mass 10.4080382663 -> 10.0270784284
- link neck: mass 0.482784902231 -> 0.465113785597
- link pelvis: mass 7.15341845835 -> 6.89158572223
- link right_arm: mass 1.74495037103 -> 1.68108088923
- link right_clavicular: mass 0.518326492016 -> 0.499354465648
- link right_foot: mass 0.910491316081 -> 0.877165091159
- link right_forearm: mass 1.06160792958 -> 1.02275046437
- link right_hand: mass 0.41408646156 -> 0.398929877075
- link right_shank: mass 2.80920246717 -> 2.70637873715
- link right_thigh: mass 9.16927117713 -> 8.83365326597
- link root: mass 0.001 -> 0.1
- link thoracic_spine: mass 9.32987685629 -> 8.98838038167
Joints:
- joint left_elbow_flexion: limit lower=-0.087 upper=2.47836753783 effort=75.0 velocity=1.0 -> lower=-0.0872664625997 upper=2.47836753783 effort=75.0 velocity=1.0
- joint right_elbow_flexion: limit lower=-0.087 upper=2.47836753783 effort=75.0 velocity=1.0 -> lower=-0.0872664625997 upper=2.47836753783 effort=75.0 velocity=1.0
