Commit message: Update human model with higher inertia for "virtual" bodies. Test joint order

File: xacro/human_model.xacro (robot description, xacro)
@@ -123,6 +123,6 @@
 	These "virtual" bodies must have a physical mass for the simulation to run.
 	They are represented as spheres with a virtual_mass and vitualRadius defined hereafter -->
-	<xacro:property name="virtual_mass" value="0.001" />
-	<xacro:property name="virtual_radius" value="0.01" />
+	<xacro:property name="virtual_mass" value="0.1" />
+	<xacro:property name="virtual_radius" value="0.03" />
 	<xacro:macro name="virtual_body" params="name">
 		<link name="${name}">
@@ -889,11 +889,5 @@
 		<dynamics damping="${jointDamping}" friction="${jointFriction}"/>
 	</joint>
-	<!-- Gazebo plugin for ROS Control -->
 	<!-- Note: if adding a Namespace here (other than "/"), the controller_manager should be in the same Namespace, as well as the spawner -->
-	<gazebo>
-		<plugin name="gazebo_ros_control" filename="libgazebo_ros_control.so">
-		<robotNamespace>/dhm</robotNamespace>
-		</plugin>
-	</gazebo>
 	<gazebo reference="root">
 		<turnGravityOff> 1 </turnGravityOff>
@@ -1057,8 +1051,8 @@
 		<type>transmission_interface/SimpleTransmission</type>
 		<joint name="lumbarspine_abduction">
-			<hardwareInterface>hardware_interface/EffortJointInterface</hardwareInterface>
+			      <hardwareInterface>EffortJointInterface</hardwareInterface>	 <hardwareInterface>PositionJointInterface</hardwareInterface>
 		</joint>
 		<actuator name="motor_lumbarspine_abduction">
-			<hardwareInterface>hardware_interface/EffortJointInterface</hardwareInterface>
+			      <hardwareInterface>EffortJointInterface</hardwareInterface>	 <hardwareInterface>PositionJointInterface</hardwareInterface>
 			<mechanicalReduction>1</mechanicalReduction>
 		</actuator>
@@ -1067,8 +1061,8 @@
 		<type>transmission_interface/SimpleTransmission</type>
 		<joint name="lumbarspine_flexion">
-			<hardwareInterface>hardware_interface/EffortJointInterface</hardwareInterface>
+			      <hardwareInterface>EffortJointInterface</hardwareInterface>	 <hardwareInterface>PositionJointInterface</hardwareInterface>
 		</joint>
 		<actuator name="motor_lumbarspine_flexion">
-			<hardwareInterface>hardware_interface/EffortJointInterface</hardwareInterface>
+			      <hardwareInterface>EffortJointInterface</hardwareInterface>	 <hardwareInterface>PositionJointInterface</hardwareInterface>
 			<mechanicalReduction>1</mechanicalReduction>
 		</actuator>
@@ -1077,8 +1071,8 @@
 		<type>transmission_interface/SimpleTransmission</type>
 		<joint name="lumbarspine_rotation">
-			<hardwareInterface>hardware_interface/EffortJointInterface</hardwareInterface>
+			      <hardwareInterface>EffortJointInterface</hardwareInterface>	 <hardwareInterface>PositionJointInterface</hardwareInterface>
 		</joint>
 		<actuator name="motor_lumbarspine_rotation">
-			<hardwareInterface>hardware_interface/EffortJointInterface</hardwareInterface>
+			      <hardwareInterface>EffortJointInterface</hardwareInterface>	 <hardwareInterface>PositionJointInterface</hardwareInterface>
 			<mechanicalReduction>1</mechanicalReduction>
 		</actuator>
@@ -1087,8 +1081,8 @@
 		<type>transmission_interface/SimpleTransmission</type>
 		<joint name="thoracicspine_abduction">
-			<hardwareInterface>hardware_interface/EffortJointInterface</hardwareInterface>
+			      <hardwareInterface>EffortJointInterface</hardwareInterface>	 <hardwareInterface>PositionJointInterface</hardwareInterface>
 		</joint>
 		<actuator name="motor_thoracicspine_abduction">
-			<hardwareInterface>hardware_interface/EffortJointInterface</hardwareInterface>
+			      <hardwareInterface>EffortJointInterface</hardwareInterface>	 <hardwareInterface>PositionJointInterface</hardwareInterface>
 			<mechanicalReduction>1</mechanicalReduction>
 		</actuator>
@@ -1097,8 +1091,8 @@
 		<type>transmission_interface/SimpleTransmission</type>
 		<joint name="thoracicspine_flexion">
-			<hardwareInterface>hardware_interface/EffortJointInterface</hardwareInterface>
+			      <hardwareInterface>EffortJointInterface</hardwareInterface>	 <hardwareInterface>PositionJointInterface</hardwareInterface>
 		</joint>
 		<actuator name="motor_thoracicspine_flexion">
-			<hardwareInterface>hardware_interface/EffortJointInterface</hardwareInterface>
+			      <hardwareInterface>EffortJointInterface</hardwareInterface>	 <hardwareInterface>PositionJointInterface</hardwareInterface>
 			<mechanicalReduction>1</mechanicalReduction>
 		</actuator>
@@ -1107,8 +1101,8 @@
 		<type>transmission_interface/SimpleTransmission</type>
 		<joint name="thoracicspine_rotation">
-			<hardwareInterface>hardware_interface/EffortJointInterface</hardwareInterface>
+			      <hardwareInterface>EffortJointInterface</hardwareInterface>	 <hardwareInterface>PositionJointInterface</hardwareInterface>
 		</joint>
 		<actuator name="motor_thoracicspine_rotation">
-			<hardwareInterface>hardware_interface/EffortJointInterface</hardwareInterface>
+			      <hardwareInterface>EffortJointInterface</hardwareInterface>	 <hardwareInterface>PositionJointInterface</hardwareInterface>
 			<mechanicalReduction>1</mechanicalReduction>
 		</actuator>
@@ -1117,8 +1111,8 @@
 		<type>transmission_interface/SimpleTransmission</type>
 		<joint name="neck_abduction">
-			<hardwareInterface>hardware_interface/EffortJointInterface</hardwareInterface>
+			      <hardwareInterface>EffortJointInterface</hardwareInterface>	 <hardwareInterface>PositionJointInterface</hardwareInterface>
 		</joint>
 		<actuator name="motor_neck_abduction">
-			<hardwareInterface>hardware_interface/EffortJointInterface</hardwareInterface>
+			      <hardwareInterface>EffortJointInterface</hardwareInterface>	 <hardwareInterface>PositionJointInterface</hardwareInterface>
 			<mechanicalReduction>1</mechanicalReduction>
 		</actuator>
@@ -1127,8 +1121,8 @@
 		<type>transmission_interface/SimpleTransmission</type>
 		<joint name="neck_flexion">
-			<hardwareInterface>hardware_interface/EffortJointInterface</hardwareInterface>
+			      <hardwareInterface>EffortJointInterface</hardwareInterface>	 <hardwareInterface>PositionJointInterface</hardwareInterface>
 		</joint>
 		<actuator name="motor_neck_flexion">
-			<hardwareInterface>hardware_interface/EffortJointInterface</hardwareInterface>
+			      <hardwareInterface>EffortJointInterface</hardwareInterface>	 <hardwareInterface>PositionJointInterface</hardwareInterface>
 			<mechanicalReduction>1</mechanicalReduction>
 		</actuator>
@@ -1137,8 +1131,8 @@
 		<type>transmission_interface/SimpleTransmission</type>
 		<joint name="neck_rotation">
-			<hardwareInterface>hardware_interface/EffortJointInterface</hardwareInterface>
+			      <hardwareInterface>EffortJointInterface</hardwareInterface>	 <hardwareInterface>PositionJointInterface</hardwareInterface>
 		</joint>
 		<actuator name="motor_neck_rotation">
-			<hardwareInterface>hardware_interface/EffortJointInterface</hardwareInterface>
+			      <hardwareInterface>EffortJointInterface</hardwareInterface>	 <hardwareInterface>PositionJointInterface</hardwareInterface>
 			<mechanicalReduction>1</mechanicalReduction>
 		</actuator>
@@ -1147,8 +1141,8 @@
 		<type>transmission_interface/SimpleTransmission</type>
 		<joint name="head_abduction">
-			<hardwareInterface>hardware_interface/EffortJointInterface</hardwareInterface>
+			      <hardwareInterface>EffortJointInterface</hardwareInterface>	 <hardwareInterface>PositionJointInterface</hardwareInterface>
 		</joint>
 		<actuator name="motor_head_abduction">
-			<hardwareInterface>hardware_interface/EffortJointInterface</hardwareInterface>
+			      <hardwareInterface>EffortJointInterface</hardwareInterface>	 <hardwareInterface>PositionJointInterface</hardwareInterface>
 			<mechanicalReduction>1</mechanicalReduction>
 		</actuator>
@@ -1157,8 +1151,8 @@
 		<type>transmission_interface/SimpleTransmission</type>
 		<joint name="head_flexion">
-			<hardwareInterface>hardware_interface/EffortJointInterface</hardwareInterface>
+			      <hardwareInterface>EffortJointInterface</hardwareInterface>	 <hardwareInterface>PositionJointInterface</hardwareInterface>
 		</joint>
 		<actuator name="motor_head_flexion">
-			<hardwareInterface>hardware_interface/EffortJointInterface</hardwareInterface>
+			      <hardwareInterface>EffortJointInterface</hardwareInterface>	 <hardwareInterface>PositionJointInterface</hardwareInterface>
 			<mechanicalReduction>1</mechanicalReduction>
 		</actuator>
@@ -1167,8 +1161,8 @@
 		<type>transmission_interface/SimpleTransmission</type>
 		<joint name="right_clavicular_flexion">
-			<hardwareInterface>hardware_interface/EffortJointInterface</hardwareInterface>
+			      <hardwareInterface>EffortJointInterface</hardwareInterface>	 <hardwareInterface>PositionJointInterface</hardwareInterface>
 		</joint>
 		<actuator name="motor_right_clavicular_flexion">
-			<hardwareInterface>hardware_interface/EffortJointInterface</hardwareInterface>
+			      <hardwareInterface>EffortJointInterface</hardwareInterface>	 <hardwareInterface>PositionJointInterface</hardwareInterface>
 			<mechanicalReduction>1</mechanicalReduction>
 		</actuator>
@@ -1177,8 +1171,8 @@
 		<type>transmission_interface/SimpleTransmission</type>
 		<joint name="right_clavicular_abduction">
-			<hardwareInterface>hardware_interface/EffortJointInterface</hardwareInterface>
+			      <hardwareInterface>EffortJointInterface</hardwareInterface>	 <hardwareInterface>PositionJointInterface</hardwareInterface>
 		</joint>
 		<actuator name="motor_right_clavicular_abduction">
-			<hardwareInterface>hardware_interface/EffortJointInterface</hardwareInterface>
+			      <hardwareInterface>EffortJointInterface</hardwareInterface>	 <hardwareInterface>PositionJointInterface</hardwareInterface>
 			<mechanicalReduction>1</mechanicalReduction>
 		</actuator>
@@ -1187,8 +1181,8 @@
 		<type>transmission_interface/SimpleTransmission</type>
 		<joint name="right_shoulder_abduction">
-			<hardwareInterface>hardware_interface/EffortJointInterface</hardwareInterface>
+			      <hardwareInterface>EffortJointInterface</hardwareInterface>	 <hardwareInterface>PositionJointInterface</hardwareInterface>
 		</joint>
 		<actuator name="motor_right_shoulder_abduction">
-			<hardwareInterface>hardware_interface/EffortJointInterface</hardwareInterface>
+			      <hardwareInterface>EffortJointInterface</hardwareInterface>	 <hardwareInterface>PositionJointInterface</hardwareInterface>
 			<mechanicalReduction>1</mechanicalReduction>
 		</actuator>
@@ -1197,8 +1191,8 @@
 		<type>transmission_interface/SimpleTransmission</type>
 		<joint name="right_shoulder_rotation">
-			<hardwareInterface>hardware_interface/EffortJointInterface</hardwareInterface>
+			      <hardwareInterface>EffortJointInterface</hardwareInterface>	 <hardwareInterface>PositionJointInterface</hardwareInterface>
 		</joint>
 		<actuator name="motor_right_shoulder_rotation">
-			<hardwareInterface>hardware_interface/EffortJointInterface</hardwareInterface>
+			      <hardwareInterface>EffortJointInterface</hardwareInterface>	 <hardwareInterface>PositionJointInterface</hardwareInterface>
 			<mechanicalReduction>1</mechanicalReduction>
 		</actuator>
@@ -1207,8 +1201,8 @@
 		<type>transmission_interface/SimpleTransmission</type>
 		<joint name="right_shoulder_flexion">
-			<hardwareInterface>hardware_interface/EffortJointInterface</hardwareInterface>
+			      <hardwareInterface>EffortJointInterface</hardwareInterface>	 <hardwareInterface>PositionJointInterface</hardwareInterface>
 		</joint>
 		<actuator name="motor_right_shoulder_flexion">
-			<hardwareInterface>hardware_interface/EffortJointInterface</hardwareInterface>
+			      <hardwareInterface>EffortJointInterface</hardwareInterface>	 <hardwareInterface>PositionJointInterface</hardwareInterface>
 			<mechanicalReduction>1</mechanicalReduction>
 		</actuator>
@@ -1217,8 +1211,8 @@
 		<type>transmission_interface/SimpleTransmission</type>
 		<joint name="right_elbow_flexion">
-			<hardwareInterface>hardware_interface/EffortJointInterface</hardwareInterface>
+			      <hardwareInterface>EffortJointInterface</hardwareInterface>	 <hardwareInterface>PositionJointInterface</hardwareInterface>
 		</joint>
 		<actuator name="motor_right_elbow_flexion">
-			<hardwareInterface>hardware_interface/EffortJointInterface</hardwareInterface>
+			      <hardwareInterface>EffortJointInterface</hardwareInterface>	 <hardwareInterface>PositionJointInterface</hardwareInterface>
 			<mechanicalReduction>1</mechanicalReduction>
 		</actuator>
@@ -1227,8 +1221,8 @@
 		<type>transmission_interface/SimpleTransmission</type>
 		<joint name="right_elbow_rotation">
-			<hardwareInterface>hardware_interface/EffortJointInterface</hardwareInterface>
+			      <hardwareInterface>EffortJointInterface</hardwareInterface>	 <hardwareInterface>PositionJointInterface</hardwareInterface>
 		</joint>
 		<actuator name="motor_right_elbow_rotation">
-			<hardwareInterface>hardware_interface/EffortJointInterface</hardwareInterface>
+			      <hardwareInterface>EffortJointInterface</hardwareInterface>	 <hardwareInterface>PositionJointInterface</hardwareInterface>
 			<mechanicalReduction>1</mechanicalReduction>
 		</actuator>
@@ -1237,8 +1231,8 @@
 		<type>transmission_interface/SimpleTransmission</type>
 		<joint name="right_wrist_flexion">
-			<hardwareInterface>hardware_interface/EffortJointInterface</hardwareInterface>
+			      <hardwareInterface>EffortJointInterface</hardwareInterface>	 <hardwareInterface>PositionJointInterface</hardwareInterface>
 		</joint>
 		<actuator name="motor_right_wrist_flexion">
-			<hardwareInterface>hardware_interface/EffortJointInterface</hardwareInterface>
+			      <hardwareInterface>EffortJointInterface</hardwareInterface>	 <hardwareInterface>PositionJointInterface</hardwareInterface>
 			<mechanicalReduction>1</mechanicalReduction>
 		</actuator>
@@ -1247,8 +1241,8 @@
 		<type>transmission_interface/SimpleTransmission</type>
 		<joint name="right_wrist_abduction">
-			<hardwareInterface>hardware_interface/EffortJointInterface</hardwareInterface>
+			      <hardwareInterface>EffortJointInterface</hardwareInterface>	 <hardwareInterface>PositionJointInterface</hardwareInterface>
 		</joint>
 		<actuator name="motor_right_wrist_abduction">
-			<hardwareInterface>hardware_interface/EffortJointInterface</hardwareInterface>
+			      <hardwareInterface>EffortJointInterface</hardwareInterface>	 <hardwareInterface>PositionJointInterface</hardwareInterface>
 			<mechanicalReduction>1</mechanicalReduction>
 		</actuator>
@@ -1257,8 +1251,8 @@
 		<type>transmission_interface/SimpleTransmission</type>
 		<joint name="left_clavicular_flexion">
-			<hardwareInterface>hardware_interface/EffortJointInterface</hardwareInterface>
+			      <hardwareInterface>EffortJointInterface</hardwareInterface>	 <hardwareInterface>PositionJointInterface</hardwareInterface>
 		</joint>
 		<actuator name="motor_left_clavicular_flexion">
-			<hardwareInterface>hardware_interface/EffortJointInterface</hardwareInterface>
+			      <hardwareInterface>EffortJointInterface</hardwareInterface>	 <hardwareInterface>PositionJointInterface</hardwareInterface>
 			<mechanicalReduction>1</mechanicalReduction>
 		</actuator>
@@ -1267,8 +1261,8 @@
 		<type>transmission_interface/SimpleTransmission</type>
 		<joint name="left_clavicular_abduction">
-			<hardwareInterface>hardware_interface/EffortJointInterface</hardwareInterface>
+			      <hardwareInterface>EffortJointInterface</hardwareInterface>	 <hardwareInterface>PositionJointInterface</hardwareInterface>
 		</joint>
 		<actuator name="motor_left_clavicular_abduction">
-			<hardwareInterface>hardware_interface/EffortJointInterface</hardwareInterface>
+			      <hardwareInterface>EffortJointInterface</hardwareInterface>	 <hardwareInterface>PositionJointInterface</hardwareInterface>
 			<mechanicalReduction>1</mechanicalReduction>
 		</actuator>
@@ -1277,8 +1271,8 @@
 		<type>transmission_interface/SimpleTransmission</type>
 		<joint name="left_shoulder_abduction">
-			<hardwareInterface>hardware_interface/EffortJointInterface</hardwareInterface>
+			      <hardwareInterface>EffortJointInterface</hardwareInterface>	 <hardwareInterface>PositionJointInterface</hardwareInterface>
 		</joint>
 		<actuator name="motor_left_shoulder_abduction">
-			<hardwareInterface>hardware_interface/EffortJointInterface</hardwareInterface>
+			      <hardwareInterface>EffortJointInterface</hardwareInterface>	 <hardwareInterface>PositionJointInterface</hardwareInterface>
 			<mechanicalReduction>1</mechanicalReduction>
 		</actuator>
@@ -1287,8 +1281,8 @@
 		<type>transmission_interface/SimpleTransmission</type>
 		<joint name="left_shoulder_rotation">
-			<hardwareInterface>hardware_interface/EffortJointInterface</hardwareInterface>
+			      <hardwareInterface>EffortJointInterface</hardwareInterface>	 <hardwareInterface>PositionJointInterface</hardwareInterface>
 		</joint>
 		<actuator name="motor_left_shoulder_rotation">
-			<hardwareInterface>hardware_interface/EffortJointInterface</hardwareInterface>
+			      <hardwareInterface>EffortJointInterface</hardwareInterface>	 <hardwareInterface>PositionJointInterface</hardwareInterface>
 			<mechanicalReduction>1</mechanicalReduction>
 		</actuator>
@@ -1297,8 +1291,8 @@
 		<type>transmission_interface/SimpleTransmission</type>
 		<joint name="left_shoulder_flexion">
-			<hardwareInterface>hardware_interface/EffortJointInterface</hardwareInterface>
+			      <hardwareInterface>EffortJointInterface</hardwareInterface>	 <hardwareInterface>PositionJointInterface</hardwareInterface>
 		</joint>
 		<actuator name="motor_left_shoulder_flexion">
-			<hardwareInterface>hardware_interface/EffortJointInterface</hardwareInterface>
+			      <hardwareInterface>EffortJointInterface</hardwareInterface>	 <hardwareInterface>PositionJointInterface</hardwareInterface>
 			<mechanicalReduction>1</mechanicalReduction>
 		</actuator>
@@ -1307,8 +1301,8 @@
 		<type>transmission_interface/SimpleTransmission</type>
 		<joint name="left_elbow_flexion">
-			<hardwareInterface>hardware_interface/EffortJointInterface</hardwareInterface>
+			      <hardwareInterface>EffortJointInterface</hardwareInterface>	 <hardwareInterface>PositionJointInterface</hardwareInterface>
 		</joint>
 		<actuator name="motor_left_elbow_flexion">
-			<hardwareInterface>hardware_interface/EffortJointInterface</hardwareInterface>
+			      <hardwareInterface>EffortJointInterface</hardwareInterface>	 <hardwareInterface>PositionJointInterface</hardwareInterface>
 			<mechanicalReduction>1</mechanicalReduction>
 		</actuator>
@@ -1317,8 +1311,8 @@
 		<type>transmission_interface/SimpleTransmission</type>
 		<joint name="left_elbow_rotation">
-			<hardwareInterface>hardware_interface/EffortJointInterface</hardwareInterface>
+			      <hardwareInterface>EffortJointInterface</hardwareInterface>	 <hardwareInterface>PositionJointInterface</hardwareInterface>
 		</joint>
 		<actuator name="motor_left_elbow_rotation">
-			<hardwareInterface>hardware_interface/EffortJointInterface</hardwareInterface>
+			      <hardwareInterface>EffortJointInterface</hardwareInterface>	 <hardwareInterface>PositionJointInterface</hardwareInterface>
 			<mechanicalReduction>1</mechanicalReduction>
 		</actuator>
@@ -1327,8 +1321,8 @@
 		<type>transmission_interface/SimpleTransmission</type>
 		<joint name="left_wrist_flexion">
-			<hardwareInterface>hardware_interface/EffortJointInterface</hardwareInterface>
+			      <hardwareInterface>EffortJointInterface</hardwareInterface>	 <hardwareInterface>PositionJointInterface</hardwareInterface>
 		</joint>
 		<actuator name="motor_left_wrist_flexion">
-			<hardwareInterface>hardware_interface/EffortJointInterface</hardwareInterface>
+			      <hardwareInterface>EffortJointInterface</hardwareInterface>	 <hardwareInterface>PositionJointInterface</hardwareInterface>
 			<mechanicalReduction>1</mechanicalReduction>
 		</actuator>
@@ -1337,8 +1331,8 @@
 		<type>transmission_interface/SimpleTransmission</type>
 		<joint name="left_wrist_abduction">
-			<hardwareInterface>hardware_interface/EffortJointInterface</hardwareInterface>
+			      <hardwareInterface>EffortJointInterface</hardwareInterface>	 <hardwareInterface>PositionJointInterface</hardwareInterface>
 		</joint>
 		<actuator name="motor_left_wrist_abduction">
-			<hardwareInterface>hardware_interface/EffortJointInterface</hardwareInterface>
+			      <hardwareInterface>EffortJointInterface</hardwareInterface>	 <hardwareInterface>PositionJointInterface</hardwareInterface>
 			<mechanicalReduction>1</mechanicalReduction>
 		</actuator>
@@ -1347,8 +1341,8 @@
 		<type>transmission_interface/SimpleTransmission</type>
 		<joint name="right_hip_abduction">
-			<hardwareInterface>hardware_interface/EffortJointInterface</hardwareInterface>
+			      <hardwareInterface>EffortJointInterface</hardwareInterface>	 <hardwareInterface>PositionJointInterface</hardwareInterface>
 		</joint>
 		<actuator name="motor_right_hip_abduction">
-			<hardwareInterface>hardware_interface/EffortJointInterface</hardwareInterface>
+			      <hardwareInterface>EffortJointInterface</hardwareInterface>	 <hardwareInterface>PositionJointInterface</hardwareInterface>
 			<mechanicalReduction>1</mechanicalReduction>
 		</actuator>
@@ -1357,8 +1351,8 @@
 		<type>transmission_interface/SimpleTransmission</type>
 		<joint name="right_hip_rotation">
-			<hardwareInterface>hardware_interface/EffortJointInterface</hardwareInterface>
+			      <hardwareInterface>EffortJointInterface</hardwareInterface>	 <hardwareInterface>PositionJointInterface</hardwareInterface>
 		</joint>
 		<actuator name="motor_right_hip_rotation">
-			<hardwareInterface>hardware_interface/EffortJointInterface</hardwareInterface>
+			      <hardwareInterface>EffortJointInterface</hardwareInterface>	 <hardwareInterface>PositionJointInterface</hardwareInterface>
 			<mechanicalReduction>1</mechanicalReduction>
 		</actuator>
@@ -1367,8 +1361,8 @@
 		<type>transmission_interface/SimpleTransmission</type>
 		<joint name="right_hip_flexion">
-			<hardwareInterface>hardware_interface/EffortJointInterface</hardwareInterface>
+			      <hardwareInterface>EffortJointInterface</hardwareInterface>	 <hardwareInterface>PositionJointInterface</hardwareInterface>
 		</joint>
 		<actuator name="motor_right_hip_flexion">
-			<hardwareInterface>hardware_interface/EffortJointInterface</hardwareInterface>
+			      <hardwareInterface>EffortJointInterface</hardwareInterface>	 <hardwareInterface>PositionJointInterface</hardwareInterface>
 			<mechanicalReduction>1</mechanicalReduction>
 		</actuator>
@@ -1377,8 +1371,8 @@
 		<type>transmission_interface/SimpleTransmission</type>
 		<joint name="right_knee_rotation">
-			<hardwareInterface>hardware_interface/EffortJointInterface</hardwareInterface>
+			      <hardwareInterface>EffortJointInterface</hardwareInterface>	 <hardwareInterface>PositionJointInterface</hardwareInterface>
 		</joint>
 		<actuator name="motor_right_knee_rotation">
-			<hardwareInterface>hardware_interface/EffortJointInterface</hardwareInterface>
+			      <hardwareInterface>EffortJointInterface</hardwareInterface>	 <hardwareInterface>PositionJointInterface</hardwareInterface>
 			<mechanicalReduction>1</mechanicalReduction>
 		</actuator>
@@ -1387,8 +1381,8 @@
 		<type>transmission_interface/SimpleTransmission</type>
 		<joint name="right_knee_flexion">
-			<hardwareInterface>hardware_interface/EffortJointInterface</hardwareInterface>
+			      <hardwareInterface>EffortJointInterface</hardwareInterface>	 <hardwareInterface>PositionJointInterface</hardwareInterface>
 		</joint>
 		<actuator name="motor_right_knee_flexion">
-			<hardwareInterface>hardware_interface/EffortJointInterface</hardwareInterface>
+			      <hardwareInterface>EffortJointInterface</hardwareInterface>	 <hardwareInterface>PositionJointInterface</hardwareInterface>
 			<mechanicalReduction>1</mechanicalReduction>
 		</actuator>
@@ -1397,8 +1391,8 @@
 		<type>transmission_interface/SimpleTransmission</type>
 		<joint name="right_ankle_flexion">
-			<hardwareInterface>hardware_interface/EffortJointInterface</hardwareInterface>
+			      <hardwareInterface>EffortJointInterface</hardwareInterface>	 <hardwareInterface>PositionJointInterface</hardwareInterface>
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