Commit message: Update human model and test

File: urdf/human_model_fixed_base.urdf (robot description, URDF)
Before this commit: robot hooman, 46 links, 45 joints
Links:
- link root: mass 0.1 -> None

File: xacro/human_model.xacro (robot description, xacro)
@@ -541,94 +541,94 @@
 	</joint>
 	<!-- Back joints -->
-	<joint name="lumbarspine_abduction" type="revolute">
+	<joint name="lumbarspine_Y" type="revolute">
 		<parent link="pelvis"/>
 		<child link="body_L5_1"/>
-		<axis xyz="1 0 0"/>
+		<axis xyz="0 1 0"/>
 		<origin xyz="0 ${S5_L5} 0"/>
-		<limit effort="${155*forceCapacity}" lower="${-15*PI/180}" upper="${15*PI/180}" velocity="${maxVelJoint}"/>
-		<dynamics damping="${jointDamping}" friction="${jointFriction}"/>
-	</joint>
-	<joint name="lumbarspine_rotation" type="revolute">
+		<limit effort="${65*forceCapacity}" lower="${-20*PI/180}" upper="${20*PI/180}" velocity="${maxVelJoint}"/>
+		<dynamics damping="${jointDamping}" friction="${jointFriction}"/>
+	</joint>
+	<joint name="lumbarspine_Z" type="revolute">
 		<parent link="body_L5_1"/>
 		<child link="body_L5_2"/>
-		<axis xyz="0 1 0"/>
-		<origin xyz="0 0 0"/>
-		<limit effort="${65*forceCapacity}" lower="${-20*PI/180}" upper="${20*PI/180}" velocity="${maxVelJoint}"/>
-		<dynamics damping="${jointDamping}" friction="${jointFriction}"/>
-	</joint>
-	<joint name="lumbarspine_flexion" type="revolute">
+		<axis xyz="0 0 1"/>
+		<origin xyz="0 0 0"/>
+		<limit effort="${228*forceCapacity}" lower="${-25*PI/180}" upper="${10*PI/180}" velocity="${maxVelJoint}"/>
+		<dynamics damping="${jointDamping}" friction="${jointFriction}"/>
+	</joint>
+	<joint name="lumbarspine_X" type="revolute">
 		<parent link="body_L5_2"/>
 		<child link="lumbar_spine"/>
-		<axis xyz="0 0 1"/>
-		<origin xyz="0 0 0"/>
-		<limit effort="${228*forceCapacity}" lower="${-25*PI/180}" upper="${10*PI/180}" velocity="${maxVelJoint}"/>
-		<dynamics damping="${jointDamping}" friction="${jointFriction}"/>
-	</joint>
-	<joint name="thoracicspine_abduction" type="revolute">
+		<axis xyz="1 0 0"/>
+		<origin xyz="0 0 0"/>
+		<limit effort="${155*forceCapacity}" lower="${-15*PI/180}" upper="${15*PI/180}" velocity="${maxVelJoint}"/>
+		<dynamics damping="${jointDamping}" friction="${jointFriction}"/>
+	</joint>
+	<joint name="thoracicspine_Y" type="revolute">
 		<parent link="lumbar_spine"/>
 		<child link="body_T12_1"/>
-		<axis xyz="1 0 0"/>
+		<axis xyz="0 1 0"/>
 		<origin xyz="0 ${L5_T12} 0"/>
-		<limit effort="${155*forceCapacity}" lower="${-15*PI/180}" upper="${15*PI/180}" velocity="${maxVelJoint}"/>
-		<dynamics damping="${jointDamping}" friction="${jointFriction}"/>
-	</joint>
-	<joint name="thoracicspine_rotation" type="revolute">
+		<limit effort="${65*forceCapacity}" lower="${-15*PI/180}" upper="${15*PI/180}" velocity="${maxVelJoint}"/>
+		<dynamics damping="${jointDamping}" friction="${jointFriction}"/>
+	</joint>
+	<joint name="thoracicspine_Z" type="revolute">
 		<parent link="body_T12_1"/>
 		<child link="body_T12_2"/>
-		<axis xyz="0 1 0"/>
-		<origin xyz="0 0 0"/>
-		<limit effort="${65*forceCapacity}" lower="${-15*PI/180}" upper="${15*PI/180}" velocity="${maxVelJoint}"/>
-		<dynamics damping="${jointDamping}" friction="${jointFriction}"/>
-	</joint>
-	<joint name="thoracicspine_flexion" type="revolute">
+		<axis xyz="0 0 1"/>
+		<origin xyz="0 0 0"/>
+		<limit effort="${228*forceCapacity}" lower="${-25*PI/180}" upper="${10*PI/180}" velocity="${maxVelJoint}"/>
+		<dynamics damping="${jointDamping}" friction="${jointFriction}"/>
+	</joint>
+	<joint name="thoracicspine_X" type="revolute">
 		<parent link="body_T12_2"/>
 		<child link="thoracic_spine"/>
-		<axis xyz="0 0 1"/>
-		<origin xyz="0 0 0"/>
-		<limit effort="${228*forceCapacity}" lower="${-25*PI/180}" upper="${10*PI/180}" velocity="${maxVelJoint}"/>
-		<dynamics damping="${jointDamping}" friction="${jointFriction}"/>
-	</joint>
-	<joint name="neck_abduction" type="revolute">
+		<axis xyz="1 0 0"/>
+		<origin xyz="0 0 0"/>
+		<limit effort="${155*forceCapacity}" lower="${-15*PI/180}" upper="${15*PI/180}" velocity="${maxVelJoint}"/>
+		<dynamics damping="${jointDamping}" friction="${jointFriction}"/>
+	</joint>
+	<joint name="neck_Y" type="revolute">
 		<parent link="thoracic_spine"/>
 		<child link="body_C7_1"/>
-		<axis xyz="1 0 0"/>
+		<axis xyz="0 1 0"/>
 		<origin xyz="0 ${T12_C7} 0"/>
-		<limit effort="50" lower="${-25*PI/180}" upper="${25*PI/180}" velocity="${maxVelJoint}"/>
-		<dynamics damping="${jointDamping}" friction="${jointFriction}"/>
-	</joint>
-	<joint name="neck_rotation" type="revolute">
+		<limit effort="50" lower="${-85*PI/180}" upper="${85*PI/180}" velocity="${maxVelJoint}"/>
+		<dynamics damping="${jointDamping}" friction="${jointFriction}"/>
+	</joint>
+	<joint name="neck_Z" type="revolute">
 		<parent link="body_C7_1"/>
 		<child link="body_C7_2"/>
-		<axis xyz="0 1 0"/>
-		<origin xyz="0 0 0"/>
-		<limit effort="50" lower="${-85*PI/180}" upper="${85*PI/180}" velocity="${maxVelJoint}"/>
-		<dynamics damping="${jointDamping}" friction="${jointFriction}"/>
-	</joint>
-	<joint name="neck_flexion" type="revolute">
+		<axis xyz="0 0 1"/>
+		<origin xyz="0 0 0"/>
+		<limit effort="50" lower="${-45*PI/180}" upper="${25*PI/180}" velocity="${maxVelJoint}"/>
+		<dynamics damping="${jointDamping}" friction="${jointFriction}"/>
+	</joint>
+	<joint name="neck_X" type="revolute">
 		<parent link="body_C7_2"/>
 		<child link="neck"/>
-		<axis xyz="0 0 1"/>
-		<origin xyz="0 0 0"/>
-		<limit effort="50" lower="${-45*PI/180}" upper="${25*PI/180}" velocity="${maxVelJoint}"/>
-		<dynamics damping="${jointDamping}" friction="${jointFriction}"/>
-	</joint>
-	<joint name="head_abduction" type="revolute">
+		<axis xyz="1 0 0"/>
+		<origin xyz="0 0 0"/>
+		<limit effort="50" lower="${-25*PI/180}" upper="${25*PI/180}" velocity="${maxVelJoint}"/>
+		<dynamics damping="${jointDamping}" friction="${jointFriction}"/>
+	</joint>
+	<joint name="head_Z" type="revolute">
 		<parent link="neck"/>
 		<child link="body_C1"/>
-		<axis xyz="1 0 0"/>
+		<axis xyz="0 0 1"/>
 		<origin xyz="0 ${C7_C1} 0"/>
-		<limit effort="20" lower="${-25*PI/180}" upper="${25*PI/180}" velocity="${maxVelJoint}"/>
-		<dynamics damping="${jointDamping}" friction="${jointFriction}"/>
-	</joint>
-	<joint name="head_flexion" type="revolute">
+		<limit effort="20" lower="${-40*PI/180}" upper="${25*PI/180}" velocity="${maxVelJoint}"/>
+		<dynamics damping="${jointDamping}" friction="${jointFriction}"/>
+	</joint>
+	<joint name="head_X" type="revolute">
 		<parent link="body_C1"/>
 		<child link="head"/>
-		<axis xyz="0 0 1"/>
-		<origin xyz="0 0 0"/>
-		<limit effort="20" lower="${-40*PI/180}" upper="${25*PI/180}" velocity="${maxVelJoint}"/>
+		<axis xyz="1 0 0"/>
+		<origin xyz="0 0 0"/>
+		<limit effort="20" lower="${-25*PI/180}" upper="${25*PI/180}" velocity="${maxVelJoint}"/>
 		<dynamics damping="${jointDamping}" friction="${jointFriction}"/>
 	</joint>
 	<!-- Right arm joints -->
-	<joint name="right_clavicular_flexion" type="revolute">
+	<joint name="right_clavicular_X" type="revolute">
 		<parent link="thoracic_spine"/>
 		<child link="body_CSJ_right_clavicular"/>
@@ -638,5 +638,5 @@
 		<dynamics damping="${jointDamping}" friction="${jointFriction}"/>
 	</joint>
-	<joint name="right_clavicular_abduction" type="revolute">
+	<joint name="right_clavicular_Y" type="revolute">
 		<parent link="body_CSJ_right_clavicular"/>
 		<child link="right_clavicular"/>
@@ -646,29 +646,29 @@
 		<dynamics damping="${jointDamping}" friction="${jointFriction}"/>
 	</joint>
-	<joint name="right_shoulder_abduction" type="revolute">
+	<joint name="right_shoulder_Y" type="revolute">
 		<parent link="right_clavicular"/>
 		<child link="body_right_shoulder_1"/>
-		<axis xyz="1 0 0"/>
+		<axis xyz="0 1 0"/>
 		<origin xyz="0 0 ${CSJ_shoulder}"/>
-		<limit effort="${69*forceCapacity}" lower="${-134*PI/180}" upper="${48*PI/180}" velocity="${maxVelJoint}"/>
-		<dynamics damping="${jointDamping}" friction="${jointFriction}"/>
-	</joint>
-	<joint name="right_shoulder_rotation" type="revolute">
+		<limit effort="${51*forceCapacity}" lower="${-34*PI/180}" upper="${97*PI/180}" velocity="${maxVelJoint}"/>
+		<dynamics damping="${jointDamping}" friction="${jointFriction}"/>
+	</joint>
+	<joint name="right_shoulder_Z" type="revolute">
 		<parent link="body_right_shoulder_1"/>
 		<child link="body_right_shoulder_2"/>
-		<axis xyz="0 1 0"/>
-		<origin xyz="0 0 0"/>
-		<limit effort="${51*forceCapacity}" lower="${-34*PI/180}" upper="${97*PI/180}" velocity="${maxVelJoint}"/>
-		<dynamics damping="${jointDamping}" friction="${jointFriction}"/>
-	</joint>
-	<joint name="right_shoulder_flexion" type="revolute">
+		<axis xyz="0 0 1"/>
+		<origin xyz="0 0 0"/>
+		<limit effort="${90*forceCapacity}" lower="${-61*PI/180}" upper="${188*PI/180}" velocity="${maxVelJoint}"/>
+		<dynamics damping="${jointDamping}" friction="${jointFriction}"/>
+	</joint>
+	<joint name="right_shoulder_X" type="revolute">
 		<parent link="body_right_shoulder_2"/>
 		<child link="right_arm"/>
-		<axis xyz="0 0 1"/>
-		<origin xyz="0 0 0"/>
-		<limit effort="${90*forceCapacity}" lower="${-61*PI/180}" upper="${188*PI/180}" velocity="${maxVelJoint}"/>
-		<dynamics damping="${jointDamping}" friction="${jointFriction}"/>
-	</joint>
-	<joint name="right_elbow_flexion" type="revolute">
+		<axis xyz="1 0 0"/>
+		<origin xyz="0 0 0"/>
+		<limit effort="${69*forceCapacity}" lower="${-134*PI/180}" upper="${48*PI/180}" velocity="${maxVelJoint}"/>
+		<dynamics damping="${jointDamping}" friction="${jointFriction}"/>
+	</joint>
+	<joint name="right_elbow_Z" type="revolute">
 		<parent link="right_arm"/>
 		<child link="body_right_elbow"/>
@@ -678,5 +678,5 @@
 		<dynamics damping="${jointDamping}" friction="${jointFriction}"/>
 	</joint>
-	<joint name="right_elbow_rotation" type="revolute">
+	<joint name="right_elbow_Y" type="revolute">
 		<parent link="body_right_elbow"/>
 		<child link="right_forearm"/>
@@ -686,5 +686,5 @@
 		<dynamics damping="${jointDamping}" friction="${jointFriction}"/>
 	</joint>
-	<joint name="right_wrist_flexion" type="revolute">
+	<joint name="right_wrist_Z" type="revolute">
 		<parent link="right_forearm"/>
 		<child link="body_right_wrist"/>
@@ -694,5 +694,5 @@
 		<dynamics damping="${jointDamping}" friction="${jointFriction}"/>
 	</joint>
-	<joint name="right_wrist_abduction" type="revolute">
+	<joint name="right_wrist_X" type="revolute">
 		<parent link="body_right_wrist"/>
 		<child link="right_hand"/>
@@ -703,5 +703,5 @@
 	</joint>
 	<!-- Left arm joints -->
-	<joint name="left_clavicular_flexion" type="revolute">
+	<joint name="left_clavicular_X" type="revolute">
 		<parent link="thoracic_spine"/>
 		<child link="body_CSJ_left_clavicular"/>
@@ -711,5 +711,5 @@
 		<dynamics damping="${jointDamping}" friction="${jointFriction}"/>
 	</joint>
-	<joint name="left_clavicular_abduction" type="revolute">
+	<joint name="left_clavicular_Y" type="revolute">
 		<parent link="body_CSJ_left_clavicular"/>
 		<child link="left_clavicular"/>
@@ -719,29 +719,29 @@
 		<dynamics damping="${jointDamping}" friction="${jointFriction}"/>
 	</joint>
-	<joint name="left_shoulder_abduction" type="revolute">
+	<joint name="left_shoulder_Y" type="revolute">
 		<parent link="left_clavicular"/>
 		<child link="body_left_shoulder_1"/>
-		<axis xyz="1 0 0"/>
+		<axis xyz="0 1 0"/>
 		<origin xyz="0 0 ${-CSJ_shoulder}"/>
-		<limit effort="${69*forceCapacity}" lower="${-48*PI/180}" upper="${134*PI/180}" velocity="${maxVelJoint}"/>
-		<dynamics damping="${jointDamping}" friction="${jointFriction}"/>
-	</joint>
-	<joint name="left_shoulder_rotation" type="revolute">
+		<limit effort="${51*forceCapacity}" lower="${-97*PI/180}" upper="${34*PI/180}" velocity="${maxVelJoint}"/>
+		<dynamics damping="${jointDamping}" friction="${jointFriction}"/>
+	</joint>
+	<joint name="left_shoulder_Z" type="revolute">
 		<parent link="body_left_shoulder_1"/>
 		<child link="body_left_shoulder_2"/>
-		<axis xyz="0 1 0"/>
-		<origin xyz="0 0 0"/>
-		<limit effort="${51*forceCapacity}" lower="${-97*PI/180}" upper="${34*PI/180}" velocity="${maxVelJoint}"/>
-		<dynamics damping="${jointDamping}" friction="${jointFriction}"/>
-	</joint>
-	<joint name="left_shoulder_flexion" type="revolute">
+		<axis xyz="0 0 1"/>
+		<origin xyz="0 0 0"/>
+		<limit effort="${90*forceCapacity}" lower="${-61*PI/180}" upper="${188*PI/180}" velocity="${maxVelJoint}"/>
+		<dynamics damping="${jointDamping}" friction="${jointFriction}"/>
+	</joint>
+	<joint name="left_shoulder_X" type="revolute">
 		<parent link="body_left_shoulder_2"/>
 		<child link="left_arm"/>
-		<axis xyz="0 0 1"/>
-		<origin xyz="0 0 0"/>
-		<limit effort="${90*forceCapacity}" lower="${-61*PI/180}" upper="${188*PI/180}" velocity="${maxVelJoint}"/>
-		<dynamics damping="${jointDamping}" friction="${jointFriction}"/>
-	</joint>
-	<joint name="left_elbow_flexion" type="revolute">
+		<axis xyz="1 0 0"/>
+		<origin xyz="0 0 0"/>
+		<limit effort="${69*forceCapacity}" lower="${-48*PI/180}" upper="${134*PI/180}" velocity="${maxVelJoint}"/>
+		<dynamics damping="${jointDamping}" friction="${jointFriction}"/>
+	</joint>
+	<joint name="left_elbow_Z" type="revolute">
 		<parent link="left_arm"/>
 		<child link="body_left_elbow"/>
@@ -751,5 +751,5 @@
 		<dynamics damping="${jointDamping}" friction="${jointFriction}"/>
 	</joint>
-	<joint name="left_elbow_rotation" type="revolute">
+	<joint name="left_elbow_Y" type="revolute">
 		<parent link="body_left_elbow"/>
 		<child link="left_forearm"/>
@@ -759,5 +759,5 @@
 		<dynamics damping="${jointDamping}" friction="${jointFriction}"/>
 	</joint>
-	<joint name="left_wrist_flexion" type="revolute">
+	<joint name="left_wrist_Z" type="revolute">
 		<parent link="left_forearm"/>
 		<child link="body_left_wrist"/>
@@ -767,5 +767,5 @@
 		<dynamics damping="${jointDamping}" friction="${jointFriction}"/>
 	</joint>
-	<joint name="left_wrist_abduction" type="revolute">
+	<joint name="left_wrist_X" type="revolute">
 		<parent link="body_left_wrist"/>
 		<child link="left_hand"/>
@@ -776,29 +776,29 @@
 	</joint>
 	<!-- Right leg joints -->
-	<joint name="right_hip_abduction" type="revolute">
+	<joint name="right_hip_Y" type="revolute">
 		<parent link="pelvis"/>
 		<child link="body_right_hip_1"/>
-		<axis xyz="1 0 0"/>
+		<axis xyz="0 1 0"/>
 		<origin xyz="0 0 ${S5_hip_horizontal}"/>
-		<limit effort="${108*forceCapacity}" lower="${-53*PI/180}" upper="${31*PI/180}" velocity="${maxVelJoint}"/>
-		<dynamics damping="${jointDamping}" friction="${jointFriction}"/>
-	</joint>
-	<joint name="right_hip_rotation" type="revolute">
+		<limit effort="${67*forceCapacity}" lower="${-34*PI/180}" upper="${39*PI/180}" velocity="${maxVelJoint}"/>
+		<dynamics damping="${jointDamping}" friction="${jointFriction}"/>
+	</joint>
+	<joint name="right_hip_Z" type="revolute">
 		<parent link="body_right_hip_1"/>
 		<child link="body_right_hip_2"/>
-		<axis xyz="0 1 0"/>
-		<origin xyz="0 0 0"/>
-		<limit effort="${67*forceCapacity}" lower="${-34*PI/180}" upper="${39*PI/180}" velocity="${maxVelJoint}"/>
-		<dynamics damping="${jointDamping}" friction="${jointFriction}"/>
-	</joint>
-	<joint name="right_hip_flexion" type="revolute">
+		<axis xyz="0 0 1"/>
+		<origin xyz="0 0 0"/>
+		<limit effort="${186*forceCapacity}" lower="${-15*PI/180}" upper="${113*PI/180}" velocity="${maxVelJoint}"/>
+		<dynamics damping="${jointDamping}" friction="${jointFriction}"/>
+	</joint>
+	<joint name="right_hip_X" type="revolute">
 		<parent link="body_right_hip_2"/>
 		<child link="right_thigh"/>
-		<axis xyz="0 0 1"/>
-		<origin xyz="0 0 0"/>
-		<limit effort="${186*forceCapacity}" lower="${-15*PI/180}" upper="${113*PI/180}" velocity="${maxVelJoint}"/>
-		<dynamics damping="${jointDamping}" friction="${jointFriction}"/>
-	</joint>
-	<joint name="right_knee_rotation" type="revolute">
+		<axis xyz="1 0 0"/>
+		<origin xyz="0 0 0"/>
+		<limit effort="${108*forceCapacity}" lower="${-53*PI/180}" upper="${31*PI/180}" velocity="${maxVelJoint}"/>
+		<dynamics damping="${jointDamping}" friction="${jointFriction}"/>
+	</joint>
+	<joint name="right_knee_Y" type="revolute">
 		<parent link="right_thigh"/>
 		<child link="body_right_knee"/>
@@ -808,5 +808,5 @@
 		<dynamics damping="${jointDamping}" friction="${jointFriction}"/>
 	</joint>
-	<joint name="right_knee_flexion" type="revolute">
+	<joint name="right_knee_Z" type="revolute">
 		<parent link="body_right_knee"/>
 		<child link="right_shank"/>
@@ -816,46 +816,46 @@
 		<dynamics damping="${jointDamping}" friction="${jointFriction}"/>
 	</joint>
-	<joint name="right_ankle_abduction" type="revolute">
+	<joint name="right_ankle_Z" type="revolute">
 		<parent link="right_shank"/>
 		<child link="body_right_ankle"/>
-		<axis xyz="1 0 0"/>
+		<axis xyz="0 0 1"/>
 		<origin xyz="0 ${-knee_ankle} 0"/>
-		<limit effort="${29*forceCapacity}" lower="${-24*PI/180}" upper="${23*PI/180}" velocity="${maxVelJoint}"/>
-		<dynamics damping="${jointDamping}" friction="${jointFriction}"/>
-	</joint>
-	<joint name="right_ankle_flexion" type="revolute">
+		<limit effort="${123*forceCapacity}" lower="${-38*PI/180}" upper="${35*PI/180}" velocity="${maxVelJoint}"/>
+		<dynamics damping="${jointDamping}" friction="${jointFriction}"/>
+	</joint>
+	<joint name="right_ankle_X" type="revolute">
 		<parent link="body_right_ankle"/>
 		<child link="right_foot"/>
-		<axis xyz="0 0 1"/>
-		<origin xyz="0 0 0"/>
-		<limit effort="${123*forceCapacity}" lower="${-38*PI/180}" upper="${35*PI/180}" velocity="${maxVelJoint}"/>
+		<axis xyz="1 0 0"/>
+		<origin xyz="0 0 0"/>
+		<limit effort="${29*forceCapacity}" lower="${-24*PI/180}" upper="${23*PI/180}" velocity="${maxVelJoint}"/>
 		<dynamics damping="${jointDamping}" friction="${jointFriction}"/>
 	</joint>
 	<!-- Left leg joints -->
-	<joint name="left_hip_abduction" type="revolute">
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